File: AntennaPcb/_autosave-AntennaPcb.kicad_pcb (KiCad board)
At the start: 2 copper layers, 90 x 90 mm, 4 parts

Commit message: Trying to improve the schematic
Parts:
- removed the G*** at (125.0, 97.3)
- removed the G*** at (121.8, 95.4)
- added G***: LOGO, AntennaPcb:Alchemy, B.Cu at (124.3, 96.7)
- added REF**: Test_Point_Keystone_5019_Minature, Connectors_TestPoints:Test_Point_Keystone_5019_Minature, B.Cu at (114.1, 95.2)
