File: AntennaPcb/AntennaPcb.sch (KiCad schematic (older format))
At the start: 0 parts

Commit message: Recreated pcb for sanity
Parts:
- added AE1: Antenna, AntennaPcb:AntennaPatch, symbol device:Antenna
- added J1: Conn_01x02, 1909763-1:TE_1909763-1, symbol conn:Conn_01x02
Changed lines of the file:
@@
-EESchema Schematic File Version 2
-LIBS:power
-LIBS:device
-LIBS:switches
-LIBS:relays
-LIBS:motors
-LIBS:transistors
-LIBS:conn
-LIBS:linear
-LIBS:regul
-LIBS:74xx
-LIBS:cmos4000
-LIBS:adc-dac
-LIBS:memory
-LIBS:xilinx
-LIBS:microcontrollers
-LIBS:dsp
-LIBS:microchip
-LIBS:analog_switches
-LIBS:motorola
-LIBS:texas
-LIBS:intel
-LIBS:audio
-LIBS:interface
-LIBS:digital-audio
-LIBS:philips
-LIBS:display
-LIBS:cypress
-LIBS:siliconi
-LIBS:opto
-LIBS:atmel
-LIBS:contrib
-LIBS:valves
-EELAYER 25 0
+EESchema Schematic File Version 4
+LIBS:AntennaPcb-cache
+EELAYER 26 0
 EELAYER END
 $Descr A4 11693 8268
@@
 $EndDescr
 $Comp
-L GND #PWR01
+L AntennaPcb-rescue:GND #PWR01
 U 1 1 5B523AE2
 P 3550 4500
@@
 $EndComp
 $Comp
-L PWR_FLAG #FLG02
+L AntennaPcb-rescue:PWR_FLAG #FLG02
 U 1 1 5B523AF6
 P 3550 4500
@@
 	1    0    0    -1
 $EndComp
+$Comp
+L device:Antenna AE1
+U 1 1 5B5D3AE4
+P 6400 3450
+F 0 "AE1" H 6480 3441 50  0000 L CNN
+F 1 "Antenna" H 6480 3350 50  0000 L CNN
+F 2 "AntennaPcb:AntennaPatch" H 6400 3450 50  0001 C CNN
+F 3 "" H 6400 3450 50  0001 C CNN
+	1    6400 3450
+	1    0    0    -1
+$EndComp
+$Comp
+L AntennaPcb-rescue:GND #PWR02
+U 1 1 5B5D3BDA
+P 6300 3650
+F 0 "#PWR02" H 6300 3400 50  0001 C CNN
+F 1 "GND" H 6305 3477 50  0000 C CNN
+F 2 "" H 6300 3650 50  0001 C CNN
+F 3 "" H 6300 3650 50  0001 C CNN
+	1    6300 3650
+	-1   0    0    1
+$EndComp
+$Comp
+L conn:Conn_01x02 J1
+U 1 1 5B5D3D4D
+P 6400 3850
+F 0 "J1" V 6273 3930 50  0000 L CNN
+F 1 "Conn_01x02" V 6364 3930 50  0000 L CNN
+F 2 "1909763-1:TE_1909763-1" H 6400 3850 50  0001 C CNN
+F 3 "~" H 6400 3850 50  0001 C CNN
+	1    6400 3850
+	0    1    1    0
+$EndComp
 $EndSCHEMATC
