File: AntennaPcb/AntennaPcb.kicad_pcb (KiCad board)
At the start: 2 copper layers, 90 x 90 mm, 2 parts

Commit message: Trying to improve the schematic
Parts:
- added G***: LOGO, AntennaPcb:Alchemy, B.Cu at (124.3, 96.7)
- added REF**: Test_Point_Keystone_5019_Minature, Connectors_TestPoints:Test_Point_Keystone_5019_Minature, B.Cu at (114.2, 95.2)
- added REF**: Test_Point_Keystone_5019_Minature, Connectors_TestPoints:Test_Point_Keystone_5019_Minature, F.Cu at (116.3, 95.5)

Commit message: Recreated pcb for sanity
Parts:
- removed the REF** at (124.5, 96.5)
- removed the REF** at (110.2, 95.2)
- removed the REF** at (114.2, 95.2)
- removed the REF** at (116.3, 95.5)
- added AE1: Antenna, AntennaPcb:AntennaPatch, F.Cu at (124.6, 94.9)
- added J1: Conn_01x02, 1909763-1:TE_1909763-1, B.Cu at (110.6, 98.1)
- added REF**: 1pin, Connectors:1pin, F.Cu at (164.5, 57.1)
- added REF**: 1pin, Connectors:1pin, F.Cu at (84.5, 57.1)
- added REF**: 1pin, Connectors:1pin, F.Cu at (84.5, 137.2)
- added REF**: 1pin, Connectors:1pin, F.Cu at (164.5, 137.2)
Routing:
- net Net-(AE1-Pad1): vias 0 -> 1

Commit message: Updating files
Other:
- board text added: "In Loving Memory"
- board text added: "of Bruce"
Changed lines of the file:
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@@
   (general
     (thickness 1.6)
-    (drawings 4)
+    (drawings 6)
     (tracks 1)
     (zones 0)
@@
     (pad 1 thru_hole circle (at 0 0) (size 4.064 4.064) (drill 3.048) (layers *.Cu *.Mask))
   )
+  (gr_text "of Bruce" (at 124.46 95.504) (layer F.SilkS)
+    (effects (font (size 1 1) (thickness 0.25)))
+  )
+  (gr_text "In Loving Memory " (at 124.968 93.472) (layer F.SilkS)
+    (effects (font (size 1 1) (thickness 0.25)))
+  )
   (gr_line (start 169.60152 141.913524) (end 169.60152 51.910482) (layer Edge.Cuts) (width 0.1))
